File: SimpleMelt-Hardware.kicad_sch (KiCad schematic)
At the start: 65 parts, among them J4 Conn_01x01, J5 Conn_01x01, J6 Conn_01x01, J7 Conn_01x01, J8 Conn_01x06, Q50 SS8050, Q51 SS8050, SW1 boot, SW2 reset, U1 ESP32-S2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

Commit message: Initial board layout completed + initial routing started
Parts:
- removed J4, J5, J6, J7: Conn_01x01, lib_fp:TGD-antenna-THT, symbol Connector_Generic:Conn_01x01
- removed J8: Conn_01x06, Connector_PinHeader_2.54mm:PinHeader_1x06_P2.54mm_Vertical, symbol Connector_Generic:Conn_01x06
- removed J? (x2): Conn_01x04, Connector_PinSocket_2.54mm:PinSocket_1x04_P2.54mm_Vertical, symbol Connector_Generic:Conn_01x04
- removed SW1: boot, Button_Switch_THT:SW_PUSH_6mm, symbol Switch:SW_Push
- removed SW2: reset, Button_Switch_THT:SW_PUSH_6mm, symbol Switch:SW_Push
- added D21: Z5V6, Diode_SMD:D_SOD-323_HandSoldering, symbol Diode:ZMMxx
- added J1, J2: Conn_01x02, Connector_PinHeader_2.54mm:PinHeader_1x02_P2.54mm_Vertical, symbol Connector_Generic:Conn_01x02
- added J200: SH_PPM, Connector_JST:JST_SH_SM04B-SRSS-TB_1x04-1MP_P1.00mm_Horizontal, symbol Connector_Generic:Conn_01x04
- added J201, J202: SH_LED, Connector_JST:JST_SH_SM04B-SRSS-TB_1x04-1MP_P1.00mm_Horizontal, symbol Connector_Generic:Conn_01x04
- added JP1: boot, AlfredoFootprints:TGD_SolderJumper, symbol Jumper:Jumper_2_Open
- added JP2: reset, AlfredoFootprints:TGD_SolderJumper, symbol Jumper:Jumper_2_Open
- added Q20: AO3401A, Package_TO_SOT_SMD:SOT-23, symbol Transistor_FET:AO3401A
- added R22: 10K, Resistor_SMD:R_0603_1608Metric, symbol Device:R
- D20: value B5819W -> 1N5819; footprint Diode_SMD:D_SOD-123 -> Diode_SMD:D_SOD-323_HandSoldering; LCSC C8598 -> C191023
- R52: value 2K -> 1K
- U1: footprint QFN56_ESP32_7X7_EXP -> AlfredoFootprints:ESP32-S2_QFN-56-1EP_7x7mm_P0.4mm
- U2: value Crystal_GND24 -> Crystal_ESP32
- U31: footprint lib_fp:TGD-TFLGA-16_3x3mm -> AlfredoFootprints:TGD-TFLGA-16_3x3mm
- gave numbers to parts that had none: 1
Connections:
- net +5V is gone; now on net VBUS: D20.2 (A)
- net E_EN: now also JP2.2 (B)
- net E_IO0: now also JP1.1 (A)
- net E_RXD: now also J2.1 (Pin_1)
- net E_TXD: now also J2.2 (Pin_2)
- net GND: now also J200.1 (Pin_1), J200.3 (Pin_3), J201.1 (Pin_1), J201.3 (Pin_3), J202.1 (Pin_1), J202.2 (Pin_2), JP1.2 (B), JP2.1 (A), R22.2
- net PPM_B: now also J200.2 (Pin_2)
- net PPM_F: now also J200.4 (Pin_4)
- net VCC: now also D21.1 (K), Q20.2 (S)
- net X_RX: now also J1.1 (Pin_1)
- net X_TX: now also J1.2 (Pin_2)
- net ExpressLRS-RX/X_RST: now reaches TP60.1
- new net: D21.2 (A), Q20.1 (G), R22.1
- new net: J202.3 (Pin_3), J202.4 (Pin_4), Q20.3 (D)
- new net LED1/LED_out: J201.4 (Pin_4)
- new net LED2/LED_out: J201.2 (Pin_2)
Other:
- removed sheet LED3
- sheet LED1 ports: added LED_out; removed none
- sheet LED2 ports: added LED_out; removed none
- note added: "TODO: ESP8285 wifi antenna? Select all JLC components By H3LIS accelerometers Order H3LIS accelerometers for global parts storage route board remove redundant ELRS parts Done: SR/SZ -> 1mm JST SH What programming interface/connector? how to do LEDs? support 6s (26V) "stiff" 1K pull resistors mando for RF resilance smaller XOs reverse polarity protection?"
- note removed: "SR/SZ -> 1mm JST SH What programming interface/connector? how to do LEDs? smaller XOs support 6s (26V) "stiff" 1K pull resistors mando for RF resilance remove redundant ELRS parts"
- moved on the sheet: C11, C12, C13, C14, C20, C21, C22, C23, C31, C40, D20, D40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

Commit message: All traces routed for V1
Parts:
- added R4: 7K, Resistor_SMD:R_0402_1005Metric, symbol Device:R
- added R5: 1K, Resistor_SMD:R_0402_1005Metric, symbol Device:R
Connections:
- net +3V3: now also R4.2
- net A1_CS: now also U1.17 (GPIO12)
- net A2_CS: now also U1.55 (GPIO46)
- net GND: now also R5.1
- net LED_1: now also U1.15 (GPIO10)
- net LED_2: now also U1.14 (GPIO9)
- net LED_MISC: now also U1.40 (GPIO36)
- net PPM_B: now also J200.4 (Pin_4), U1.39 (GPIO35); no longer J200.2 (Pin_2)
- net PPM_F: now also J200.2 (Pin_2), U1.38 (GPIO34); no longer J200.4 (Pin_4)
- net P_MISO: now also U1.19 (GPIO14)
- net P_MOSI: now also U1.18 (GPIO13)
- net P_SCK: now also U1.16 (GPIO11)
- net SNS_VIN: now also U1.8 (GPIO3)
- net X_RX: now also U1.13 (GPIO8)
- net X_TX: now also U1.12 (GPIO7)
- new net: R4.1, R5.2
Other:
- moved on the sheet: J200

Commit message: All LCSC components selected
Parts:
- removed TP60: TP_RST, AlfredoFootprints:GE_TestPoint_Loop, symbol Connector:TestPoint
- C10: LCSC ? -> C1546
- C11, C12, C22: LCSC ? -> C32949
- C2, C52: LCSC ? -> C15525
- C3, C6, C9: LCSC ? -> C52923
- R1, R3, R40, R41, R5, R50, R51, R52, R53: LCSC ? -> C11702
- R2: LCSC ? -> C25123
- R22: footprint Resistor_SMD:R_0603_1608Metric -> Resistor_SMD:R_0402_1005Metric; LCSC C25804 -> C25744
- R4: LCSC ? -> C25917
- R54, R55, R56, R57: LCSC ? -> C25905
Connections:
- net at R4.1, R5.2: now also U1.28 (GPIO21)
Other:
- sheet ExpressLRS-RX ports: added none; removed X_RST
- note added: "TODO: By H3LIS accelerometers Order H3LIS accelerometers for global parts storage Eventual: remove redundant parts ESP8285 wifi antenna? Done: SR/SZ -> 1mm JST SH What programming interface/connector? how to do LEDs? support 6s (26V) "stiff" 1K pull resistors mando for RF resilance smaller XOs reverse polarity protection? route board Select all JLC components"
- note removed: "TODO: ESP8285 wifi antenna? Select all JLC components By H3LIS accelerometers Order H3LIS accelerometers for global parts storage route board remove redundant ELRS parts Done: SR/SZ -> 1mm JST SH What programming interface/connector? how to do LEDs? support 6s (26V) "stiff" 1K pull resistors mando for RF resilance smaller XOs reverse polarity protection?"
- moved on the sheet: J1, J2, J200, J201, R4, R5

Commit message: Rotini V1
Parts:
- added R6, R7, R8: 300R, Resistor_SMD:R_1206_3216Metric, symbol Device:R
Changed lines of the file:
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@@
+    (pin "2")
+  )
+  (symbol (lib_id "Device:R") (at 318.77 96.52 0) (unit 1)
+    (in_bom yes) (on_board yes) (fields_autoplaced)
+    (property "Reference" "R7" (id 0) (at 321.31 95.2499 0)
+      (effects (font (size 1.27 1.27)) (justify left))
+    )
+    (property "Value" "300R" (id 1) (at 321.31 97.7899 0)
+      (effects (font (size 1.27 1.27)) (justify left))
+    )
+    (property "Footprint" "Resistor_SMD:R_1206_3216Metric" (id 2) (at 316.992 96.52 90)
+      (effects (font (size 1.27 1.27)) hide)
+    )
+    (property "Datasheet" "https://lcsc.com/product-detail/Chip-Resistor---Surface-Mount_UNI-ROYALUniroyal-Elec-UNI-ROYALUniroyal-Elec-1206W4F3000T5E_C17887.html" (id 3) (at 318.77 96.52 0)
+      (effects (font (size 1.27 1.27)) hide)
+    )
+    (property "LCSC" "C17887" (id 4) (at 318.77 96.52 0)
+      (effects (font (size 1.27 1.27)) hide)
+    )
+    (pin "1")
     (pin "2")
   )
@@
     )
     (pin "1")
+  )
+  (symbol (lib_id "Device:R") (at 332.74 97.79 0) (unit 1)
+    (in_bom yes) (on_board yes) (fields_autoplaced)
+    (property "Reference" "R8" (id 0) (at 335.28 96.5199 0)
+      (effects (font (size 1.27 1.27)) (justify left))
+    )
+    (property "Value" "300R" (id 1) (at 335.28 99.0599 0)
+      (effects (font (size 1.27 1.27)) (justify left))
+    )
+    (property "Footprint" "Resistor_SMD:R_1206_3216Metric" (id 2) (at 330.962 97.79 90)
+      (effects (font (size 1.27 1.27)) hide)
+    )
+    (property "Datasheet" "https://lcsc.com/product-detail/Chip-Resistor---Surface-Mount_UNI-ROYALUniroyal-Elec-UNI-ROYALUniroyal-Elec-1206W4F3000T5E_C17887.html" (id 3) (at 332.74 97.79 0)
+      (effects (font (size 1.27 1.27)) hide)
+    )
+    (property "LCSC" "C17887" (id 4) (at 332.74 97.79 0)
+      (effects (font (size 1.27 1.27)) hide)
+    )
+    (pin "1")
+    (pin "2")
+  )
+  (symbol (lib_id "Device:R") (at 306.07 97.79 0) (unit 1)
+    (in_bom yes) (on_board yes) (fields_autoplaced)
+    (property "Reference" "R6" (id 0) (at 308.61 96.5199 0)
+      (effects (font (size 1.27 1.27)) (justify left))
+    )
+    (property "Value" "300R" (id 1) (at 308.61 99.0599 0)
+      (effects (font (size 1.27 1.27)) (justify left))
+    )
+    (property "Footprint" "Resistor_SMD:R_1206_3216Metric" (id 2) (at 304.292 97.79 90)
+      (effects (font (size 1.27 1.27)) hide)
+    )
+    (property "Datasheet" "https://lcsc.com/product-detail/Chip-Resistor---Surface-Mount_UNI-ROYALUniroyal-Elec-UNI-ROYALUniroyal-Elec-1206W4F3000T5E_C17887.html" (id 3) (at 306.07 97.79 0)
+      (effects (font (size 1.27 1.27)) hide)
+    )
+    (property "LCSC" "C17887" (id 4) (at 306.07 97.79 0)
+      (effects (font (size 1.27 1.27)) hide)
+    )
+    (pin "1")
+    (pin "2")
   )
   (symbol (lib_id "Device:R") (at 153.67 243.84 0) (mirror y) (unit 1)
@@
       (reference "R5") (unit 1) (value "1K") (footprint "Resistor_SMD:R_0402_1005Metric")
     )
+    (path "/77821fb9-1e5b-49ef-bf97-0705d83d07e9"
+      (reference "R6") (unit 1) (value "300R") (footprint "Resistor_SMD:R_1206_3216Metric")
+    )
+    (path "/0416b95c-33dc-4108-9a3f-fb4a00b2e2b2"
+      (reference "R7") (unit 1) (value "300R") (footprint "Resistor_SMD:R_1206_3216Metric")
+    )
+    (path "/750211bf-8a25-421d-bb9a-9a436fd3b726"
+      (reference "R8") (unit 1) (value "300R") (footprint "Resistor_SMD:R_1206_3216Metric")
+    )
     (path "/00000000-0000-0000-0000-000060dcbf0d"
