File: Rotini-Hardware/LEDdriver.kicad_sch (KiCad schematic)
At the start: 5 parts, among them Q30 LBSS84LT1G, Q31 2N7002

Commit message: changed footprints
Parts:
- Q30, Q31: footprint Package_TO_SOT_SMD:SOT-23 -> AlfredoFootprints:SOT-23-small
Changed lines of the file:
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@@
       (effects (font (size 1.27 1.27)) (justify left))
     )
-    (property "Footprint" "Package_TO_SOT_SMD:SOT-23" (at 142.24 113.665 0)
+    (property "Footprint" "AlfredoFootprints:SOT-23-small" (at 142.24 113.665 0)
       (effects (font (size 1.27 1.27) italic) (justify left) hide)
     )
@@
       (effects (font (size 1.27 1.27)) (justify left))
     )
-    (property "Footprint" "Package_TO_SOT_SMD:SOT-23" (at 156.21 94.615 0)
+    (property "Footprint" "AlfredoFootprints:SOT-23-small" (at 156.21 94.615 0)
       (effects (font (size 1.27 1.27) italic) (justify left) hide)
     )
